File: KiCAD/FreeEEG32-prealpha2.sch (KiCad schematic (older format))
At the start: 0 parts

Commit message: added usb, crystals
Parts:
- added R1, R11, R12, R13, R14, R15, R16, R17, R18, R19, R2, R20, R21, R22, R23, R24, R25, R26, R27, R28, R29, R3, R30, R31, R32, R33, R34, R4, R5, R6, R7, R8, R9: 0, Resistor_SMD:R_0402_1005Metric, symbol Device:R_Small
Connections:
- new net ADC4_22_DGND: R20.2
- new net ADC4_24_IOVDD: R19.2
- new net ADC4_31_XTAL1: R22.2, R23.2
- new net ADC4_32_XTAL2_MCLK: R21.2
- new net AVDD_1_IN: R13.2, R17.2, R8.2
- new net AVDD_2_GND: R14.2, R18.2
- new net AVDD_3_EN: R8.1
- new net CRYSTAL_2_GND: R16.1
- new net CRYSTAL_3_OUT: R21.1
- new net CRYSTAL_4_Vin: R15.1
- new net IOVDD_1_IN: R11.2, R15.2, R7.2
- new net IOVDD_2_GND: R12.2, R16.2, R20.1, R22.1, R23.1
- new net IOVDD_3_EN: R7.1
- new net IOVDD_5_OUT: R19.1
- new net MCU_103_PA11_USB_OTG_FS_DM: R2.2
- new net MCU_104_PA12_USB_OTG_FS_DP: R1.2
- new net MCU_108_VDD: R32.1
- new net MCU_121_VDDSDMMC: R33.1
- new net MCU_131_VDD: R34.1
- new net MCU_17_VDD: R24.1
- new net MCU_30_VDD: R25.1
- new net MCU_33_VDDA: R26.1
- new net MCU_39_VDD: R27.1
- new net MCU_52_VDD: R28.1
- new net MCU_62_VDD: R29.1
- new net MCU_72_VDD: R30.1
- new net MCU_84_VDD: R31.1
- new net MCU_94_VSS: R6.1
- new net MCU_95_VDDUSB: R5.1
- new net POWER_3_OUT1A2B_DIODES: R11.1, R13.1
- new net POWER_4_OUT1B2A: R12.1, R14.1
- new net REF_2_VIN: R17.1
- new net REF_4_GND: R18.1
- new net USB_1_VBUS: R3.1
- new net USB_2_D-: R2.1
- new net USB_3_D+: R1.1
- new net USB_5_GND: R4.1
- new net VDD_1_IN: R3.2, R9.2
- new net VDD_2_GND: R4.2, R6.2
- new net VDD_3_EN: R9.1
- new net VDD_5_OUT: R24.2, R25.2, R26.2, R27.2, R28.2, R29.2, R30.2, R31.2, R32.2, R33.2, R34.2, R5.2
